Commit message: Mask LiDAR rear-hemisphere artifact at the sensor, document as a stated limitation
Masked gpu_lidar to a clean +-90 deg (180 total) front FOV via new
lidar_horizontal_fov/lidar_samples xacro properties, rather than
filtering downstream - avoids a two-topics-diverge failure mode where
one consumer (e.g. AMCL) could end up reading the unfiltered scan.
Verified fully clean: 0/180 self-hits (was 176/360), rate still ~5Hz.

Confirmed exact gz-sim version (6.18.0) and searched upstream; no exact
match for this specific sensor-frame-relative symptom, closest related
is the still-open gazebosim/gz-sim#2743 (general gpu_lidar accuracy
degradation). Recorded rather than filed - filing is a public action
left for the user to decide on.

Added README.md with a stated Known Limitations section (180 LiDAR FOV
+ 8m range cap, IL-not-RL SARL checkpoint, ground-truth perception
default) so these are visible constraints, not accidents discovered
later. Updated Phase 2's plan to treat AMCL tuning and costmap
raytracing/decay as first-class tasks given the reduced FOV.

File: crowd_nav_ws/src/crowd_nav_description/urdf/nvis_3302ard.xacro (robot description, xacro)
@@ -44,11 +44,23 @@
        sensor's own rear-hemisphere rendering, NOT robot geometry - rotating the sensor's yaw
        180deg moved the artifact with it (sensor-frame-relative, not world-frame-relative),
-       and no amount of standoff height changed that. This is a gz-sim/ogre2 rendering
-       limitation on this Fortress install, not a modeling error; a CPU "lidar" sensor type
-       was tried as an alternative and found completely non-functional on this install (no
-       gz-transport topic at all). Settled back on a modest, physically-defensible 0.03 m
-       standoff (raising it further doesn't help, since the cause isn't clearance) - full
-       diagnostic trail in docs/phase1-findings.md. This is an OPEN ISSUE to resolve before
-       Phase 2 (Nav2/costmap) can produce meaningful results with a full 360deg scan. -->
+       and no amount of standoff height changed that. Confirmed as a gz-sim 6.18.0 (Fortress)
+       rendering limitation, not a modeling error - see docs/phase1-findings.md for the full
+       diagnostic trail and upstream issue search. A CPU "lidar" sensor type was tried as an
+       alternative and found completely non-functional on this install (no gz-transport topic
+       at all). Settled back on a modest, physically-defensible 0.03 m standoff (raising it
+       further doesn't help, since the cause isn't clearance). -->
+  <!-- DECISION (2026-07-22, masking chosen over a downstream filter node - see
+       docs/phase1-findings.md for the reasoning: masking at the source means there is only
+       ever one /scan topic, avoiding the failure mode where one consumer reads the filtered
+       topic and another reads the raw one): masked to the front ~180deg, safely inside the
+       measured ~184deg clean arc (2 deg margin either side). This makes the sensor
+       deliberately pessimistic in field of view on top of the already-deliberate 8 m range
+       cap (S3 of the brief) - closer to a real budget 180deg LiDAR than the original 360deg
+       spec, and that combination should be stated as a known limitation, not an accident.
+       samples scales with the FOV to hold the ~1 deg angular resolution spec (S3) constant.
+       Restore lidar_horizontal_fov to ${2*pi} (and samples to 360) in one place here if a
+       gz-sim version without this rendering bug is ever confirmed. -->
+  <xacro:property name="lidar_horizontal_fov" value="${pi}"/>
+  <xacro:property name="lidar_samples" value="180"/>
   <material name="chassis_grey">
     <color rgba="0.6 0.6 0.6 1.0"/>
@@ -155,5 +167,7 @@
     parent_link="base_link"
     xyz="0 0 ${chassis_z - axle_z + chassis_height/2.0 + lidar_standoff}"
-    rpy="0 0 0"/>
+    rpy="0 0 0"
+    horizontal_fov="${lidar_horizontal_fov}"
+    samples="${lidar_samples}"/>
   <!-- ================= ros2_control hardware interface (swap point) ================= -->
   <xacro:nvis_3302ard_ros2_control/>

Commit message: Add DDS hygiene tooling, fix robot_radius spec inconsistency
scripts/ros2_teardown.sh: graceful shutdown + safe /dev/shm cleanup,
scripts/check_dds_health.sh: fails loudly if stale FastRTPS segments
exceed a threshold, wired into spawn_robot.launch.py so a dirty
session fails the launch immediately instead of hanging 40s later.
This will matter for real once Phase 10's evaluation harness runs the
full stack unattended hundreds of times.

Added crowd_nav_onnxruntime_vendor... no wait, added
robot_collision_radius as a single-source-of-truth xacro property
(diagonal-based, 0.14m) that crowd_nav_bringup's Nav2 config now
references explicitly, and flagged as a hard requirement for Phase 9's
safety supervisor to use the same value.

Also fixed a real inconsistency caught while doing this: S4.3 of the
plan incorrectly listed the OOD proximity threshold as a robot_radius
consumer - S4.4 is explicit that it correctly uses policy_radius
instead. Corrected the plan text rather than leave the contradiction.

File: crowd_nav_ws/src/crowd_nav_description/urdf/nvis_3302ard.xacro (robot description, xacro)
@@ -9,4 +9,15 @@
   <xacro:property name="chassis_height" value="0.080"/>
   <xacro:property name="total_mass"     value="1.0"/>
+  <!-- Single source of truth for any circular collision-radius approximation of this robot
+       (Nav2 costmaps, the Phase 9 safety supervisor's forward-sim collision check - see
+       IMPLEMENTATION_PLAN.md S4.3). MUST be derived from the chassis DIAGONAL
+       (sqrt((L/2)^2+(W/2)^2) = 0.1344 m), not the smaller face-normal half-width (0.095 m) -
+       a real bug found in Phase 2 (docs/phase2-findings.md): an under-sized circular radius
+       lets a planner think a squeeze is clear when the real square corners would clip.
+       0.14 m adds a small margin over the exact 0.1344 m diagonal. Every consumer of a
+       circular robot radius should reference this value, not re-derive or hardcode its own -
+       crowd_nav_bringup/config/nav2_params.yaml's robot_radius already matches this; Phase 9
+       must too. -->
+  <xacro:property name="robot_collision_radius" value="0.14"/>
   <!-- [PENDING] ESTIMATES, to be replaced with measured values. See MEASUREMENTS.md. -->
   <xacro:property name="wheel_radius"     value="0.0325"/> <!-- [PENDING] -->

Commit message: Close Phase 2: root-cause tip-over, SLAM double-mapping, and goal overshoot
The prior session left three things open and correctly stopped rather than
paper over them. This session root-causes all three and meets the agreed
done-bar (5 consecutive NavigateToPose goals, both AMCL and SLAM modes, no
manual intervention), verified against Gazebo ground-truth pose rather than
odometry alone.

Root cause chain:
- The SLAM map's "ghost obstacle" and the AMCL chain's "unexplained overshoot"
  were both downstream of the robot physically tipping over during driving
  (~33 deg pitch, invisible to odometry). Four compounding bugs: a wheel/
  caster joint z-offset bug that buried the wheels below the floor at spawn,
  caster friction too high for in-place rotation, and - the real structural
  fix - caster_mass too small (0.02kg), leaving the caster carrying only ~2%
  of the robot's static weight by torque balance. Raised to 0.15kg (~15%
  share); acceleration limits also moderated as a secondary safety margin.
- A second, independent SLAM issue after the physics fix: fast 180/360 deg
  in-place spins combined with the deliberately-narrowed ~180 deg LiDAR FOV
  caused scan-matcher tracking loss. Fixed by retiring hand-rolled cmd_vel
  mapping scripts in favor of NavigateToPose waypoint goals, using Nav2's
  own MPPI controller and costmap planner instead of reimplementing it.
- The goal overshoot was NavFn's known near-goal degenerate-path brittleness
  recurring at a larger stall distance; xy_goal_tolerance/planner tolerance
  loosened further and kept in sync.

Full bug-by-bug diagnostic trail, including several intermediate fixes that
were necessary but not sufficient on their own, in docs/phase2-findings.md.

File: crowd_nav_ws/src/crowd_nav_description/urdf/nvis_3302ard.xacro (robot description, xacro)
@@ -35,5 +35,16 @@
        approximation for inertia purposes on a robot this size. -->
   <xacro:property name="wheel_mass"  value="0.05"/>  <!-- [PENDING], each wheel -->
-  <xacro:property name="caster_mass" value="0.02"/>  <!-- [PENDING] -->
+  <!-- caster_mass revised up from an initial 0.02 kg (docs/phase2-findings.md): that value
+       treated the caster as just the bare ball, but a real caster is an assembly (bracket +
+       swivel + ball), and more importantly, with chassis mass distributed as a symmetric box
+       centered directly over the drive-wheel axle, the system COM sits almost exactly at the
+       wheel axle (torque-balance math: COM offset from the axle is caster_mass*caster_offset_x
+       / total_mass) - at 0.02 kg the caster carried only ~2% of the robot's static weight, a
+       stability margin so thin that ordinary accel/decel transients during driving (braking
+       after forward motion, reversing turn direction) could momentarily unweight it enough to
+       tip the chassis, confirmed via ground-truth pose logging across many repro attempts.
+       0.15 kg brings that to ~15% - still physically reasonable for a caster assembly on a 1 kg
+       robot, and enough static margin that transient unweighting no longer fully lifts it. -->
+  <xacro:property name="caster_mass" value="0.15"/>  <!-- [PENDING] -->
   <xacro:property name="chassis_mass" value="${total_mass - 2*wheel_mass - caster_mass}"/>
   <!-- Wheel axle height above the ground/base_footprint plane. Derived from wheel_radius
@@ -142,6 +153,30 @@
       <parent link="base_link"/>
       <child link="${prefix}_wheel"/>
-      <origin xyz="0 ${reflect * wheel_separation/2.0} ${axle_z - chassis_z}" rpy="0 0 0"/>
+      <!-- base_link's own origin (via base_footprint_joint) is already placed at axle_z above
+           the ground, so the wheel joint needs NO further z-offset - it sits at z=0 relative to
+           base_link. A previous version used "${axle_z - chassis_z}" here (-0.03 m), which
+           re-offset the wheel relative to the CHASSIS's center height instead of relative to
+           base_link's own (already-correct) origin. That silently buried the wheels 3 cm below
+           the ground plane at spawn (while the caster, computed off the same wrong baseline,
+           ended up floating ~1 cm above it) - the physics engine's contact resolution reacted
+           to that invalid interpenetration with a large corrective torque, tipping the chassis
+           to a stable ~33 deg equilibrium within about two minutes of sim time, with the wheels
+           still spinning throughout (encoder-driven odometry kept accumulating "distance" the
+           whole time). That is what actually produced the "ghost obstacle" SLAM map corruption
+           and the huge odom-vs-ground-truth divergence chased across the v1-v4 driving-script
+           iterations (docs/phase2-findings.md) - none of those were the real bug. Confirmed via
+           a ground-truth pose monitor showing pitch grow steadily from spawn with ZERO drive
+           commands ever sent, ruling out anything in the driving scripts. -->
+      <origin xyz="0 ${reflect * wheel_separation/2.0} 0" rpy="0 0 0"/>
       <axis xyz="0 1 0"/>
+      <!-- Joint damping: a real motor/gearbox has internal damping a rigid-body sim doesn't
+           model by default. Without it, ANY sudden commanded-velocity reversal (braking after
+           forward motion, reversing turn direction, turning right after forward motion) applies
+           a near-instant torque change to a wheel, which - combined with the caster's very thin
+           static load margin, see the caster friction comment below - was enough to tip the
+           chassis. diff_drive_controller.yaml's acceleration limits address the SAME root cause
+           from the command side (see its comment) but only for the specific transition each
+           limit targets; this is the general, structural version of the same fix. -->
+      <dynamics damping="0.05" friction="0.0"/>
     </joint>
   </xacro:macro>
@@ -172,5 +207,9 @@
     <parent link="base_link"/>
     <child link="caster_wheel"/>
-    <origin xyz="${caster_offset_x} 0 ${axle_z - chassis_z + wheel_radius - caster_radius}" rpy="0 0 0"/>
+    <!-- Caster sphere's bottom should touch the ground plane, same as the wheels: center at
+         caster_radius above ground, i.e. (caster_radius - axle_z) relative to base_link's
+         origin (which sits at axle_z above ground). See the wheel joint comment above for the
+         wrong-baseline bug this replaces. -->
+    <origin xyz="${caster_offset_x} 0 ${caster_radius - axle_z}" rpy="0 0 0"/>
   </joint>
   <!-- ================= LiDAR ================= -->
@@ -191,3 +230,33 @@
     <material>Gazebo/Grey</material>
   </gazebo>
+  <!-- Caster friction: no friction coefficient was specified anywhere for this model, so the
+       physics engine's default (high enough to resist sliding) applied to the caster sphere too.
+       During any pure in-place rotation (ang!=0, lin=0 - used constantly by the SLAM coverage
+       sweep scripts, docs/phase2-findings.md), the two drive wheels spin in place while the
+       caster, offset behind the axle, needs to scrub/slide sideways to let the chassis pivot. A
+       high-friction caster can't do that smoothly - it catches, and the resulting torque tips
+       the chassis up on one side while yaw keeps climbing unbounded and x/y freezes. Confirmed
+       empirically: ground-truth pose logging showed exactly this signature (frozen position,
+       runaway yaw, pitch jumping to ~17 deg) starting mid-way through the very first in-place
+       turn segment of a sweep, on a model where the earlier wheel/caster z-offset bug (see the
+       wheel joint comment above) had already been fixed and ruled out. Near-zero friction here
+       lets the caster pivot freely, as it physically would (it's a small low-friction ball
+       caster on the real hardware, not a driven/gripping wheel). -->
+  <gazebo reference="caster_wheel">
+    <mu1>0.001</mu1>
+    <mu2>0.001</mu2>
+  </gazebo>
+  <!-- Drive wheel friction: previously left unspecified (engine default), same as the ground
+       plane's own unspecified <ode/> friction block. Set explicitly to a normal, grippy value -
+       traction is what lets the wheels roll instead of skid, including during the sudden
+       rolling-to-differential transition when a forward move is immediately followed by an
+       in-place turn. -->
+  <gazebo reference="left_wheel">
+    <mu1>1.0</mu1>
+    <mu2>1.0</mu2>
+  </gazebo>
+  <gazebo reference="right_wheel">
+    <mu1>1.0</mu1>
+    <mu2>1.0</mu2>
+  </gazebo>
 </robot>
